File: moduleur-vco/VCO/VCO_panel.kicad_pcb (KiCad board)
At the start: 2 copper layers, 252.6 x 128.5 mm, 144 parts

Commit message: Update mousebites
Parts:
- removed KiKit_MB_11_1, KiKit_MB_11_9, KiKit_MB_13_1, KiKit_MB_13_9, KiKit_MB_15_1, KiKit_MB_15_9, KiKit_MB_17_1, KiKit_MB_17_9, KiKit_MB_1_1, KiKit_MB_1_9, KiKit_MB_3_1, KiKit_MB_3_9, KiKit_MB_5_1, KiKit_MB_5_9, KiKit_MB_7_1, KiKit_MB_7_9, KiKit_MB_9_1, KiKit_MB_9_9: NPTH, NPTH
- moved KiKit_MB_11_2 4.53 mm to (124.9, 94.2)
- moved KiKit_MB_11_8 4.53 mm to (124.9, 89.8)
- moved KiKit_MB_13_2 4.53 mm to (188.9, 36.2)
- moved KiKit_MB_13_8 4.53 mm to (188.9, 31.8)
- moved KiKit_MB_15_2 4.53 mm to (188.9, 64.8)
- moved KiKit_MB_15_8 4.53 mm to (188.9, 60.2)
- moved KiKit_MB_17_2 4.53 mm to (188.9, 94.2)
- moved KiKit_MB_17_8 4.53 mm to (188.9, 89.8)
- moved KiKit_MB_1_2 4.53 mm to (60.9, 36.2)
- moved KiKit_MB_1_8 4.53 mm to (60.9, 31.8)
- moved KiKit_MB_3_2 4.53 mm to (60.9, 64.8)
- moved KiKit_MB_3_8 4.53 mm to (60.9, 60.2)
- moved KiKit_MB_5_2 4.53 mm to (60.9, 94.2)
- moved KiKit_MB_5_8 4.53 mm to (60.9, 89.8)
- moved KiKit_MB_7_2 4.53 mm to (124.9, 36.2)
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