File: VCA/VCA.kicad_pcb (KiCad board)
At the start: 2 copper layers, 252.9 x 128.5 mm, 0 parts

Commit message: Add URL and re-panelize
Other:
- board text added: "https://github.com/domesticmouse/moduleur-faceplates"
Changed lines of the file:
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@@
 		(layer "Edge.Cuts")
+	)
+	(gr_text "https://github.com/domesticmouse/moduleur-faceplates"
+		(at 28.67 38.42 90)
+		(layer "B.SilkS")
+		(effects
+			(font
+				(size 2 2)
+			)
+			(justify left bottom mirror)
+		)
+	)
+	(gr_text "https://github.com/domesticmouse/moduleur-faceplates"
+		(at 92.75 38.42 90)
+		(layer "B.SilkS")
+		(effects
+			(font
+				(size 2 2)
+			)
+			(justify left bottom mirror)
+		)
+	)
+	(gr_text "https://github.com/domesticmouse/moduleur-faceplates"
+		(at 156.56 38.42 90)
+		(layer "B.SilkS")
+		(effects
+			(font
+				(size 2 2)
+			)
+			(justify left bottom mirror)
+		)
+	)
+	(gr_text "https://github.com/domesticmouse/moduleur-faceplates"
+		(at 221.17 38.42 90)
+		(layer "B.SilkS")
+		(effects
+			(font
+				(size 2 2)
+			)
+			(justify left bottom mirror)
+		)
 	)
 	(group ""
