File: VCA/VCA_panel.kicad_pcb (KiCad board)
At the start: 2 copper layers, 252.9 x 128.5 mm, 126 parts

Commit message: Add URL and re-panelize
Other:
- board text added: "https://github.com/domesticmouse/moduleur-faceplates"
