File: VCO/VCO.kicad_pcb (KiCad board)
At the start: 2 copper layers, 252.3 x 128.5 mm, 0 parts

Commit message: Add URL and re-panelize
Other:
- board text added: "https://github.com/domesticmouse/moduleur-faceplates"
Changed lines of the file:
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@@
 		(layer "Edge.Cuts")
+	)
+	(gr_text "https://github.com/domesticmouse/moduleur-faceplates"
+		(at 27.25 66.13 90)
+		(layer "B.SilkS")
+		(effects
+			(font
+				(size 2 2)
+			)
+			(justify left bottom mirror)
+		)
+	)
+	(gr_text "https://github.com/domesticmouse/moduleur-faceplates"
+		(at 91.74 66.13 90)
+		(layer "B.SilkS")
+		(effects
+			(font
+				(size 2 2)
+			)
+			(justify left bottom mirror)
+		)
+	)
+	(gr_text "https://github.com/domesticmouse/moduleur-faceplates"
+		(at 154.96 66.13 90)
+		(layer "B.SilkS")
+		(effects
+			(font
+				(size 2 2)
+			)
+			(justify left bottom mirror)
+		)
+	)
+	(gr_text "https://github.com/domesticmouse/moduleur-faceplates"
+		(at 219.55 66.13 90)
+		(layer "B.SilkS")
+		(effects
+			(font
+				(size 2 2)
+			)
+			(justify left bottom mirror)
+		)
 	)
 	(embedded_fonts no)
